File: hardware/0.1/Hub20.sch (KiCad schematic (older format))
At the start: 126 parts, among them J1 USB_C_Receptacle_USB2.0, Q1 DTC123J, Q2 BSS138, SW1 SW_Push, SW10 MX_RGB, SW11 MX_RGB, SW12 MX_RGB, SW13 Encoder_MX_RGB, SW14 MX_RGB, SW15 MX_RGB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

Commit message: clean up routing, design review TODO
Parts:
- added LOGO5: OSHW, josh-logos:OSHW_Logo_3.6x3.6_F.Mask, symbol Mechanical:MountingHole
Connections:
- net R4: now also U3.12 (PA2); no longer U3.11 (PA1)
- net R5: now also U3.11 (PA1); no longer U3.12 (PA2)
Changed lines of the file:
@@
 R3
 Text Label 9000 3350 2    50   ~ 0
-R4
-Text Label 9000 3450 2    50   ~ 0
 R5
 Text Label 9000 3850 2    50   ~ 0
@@
 Wire Wire Line
 	9000 3250 8450 3250
-Wire Wire Line
-	9000 3350 8450 3350
-Wire Wire Line
-	9000 3450 8450 3450
 Wire Wire Line
 	9000 4250 8450 4250
@@
 NoConn ~ 7150 2550
 NoConn ~ 7150 2650
+Wire Wire Line
+	9000 3350 8450 3350
+Wire Wire Line
+	9000 3450 8450 3450
+Text Label 9000 3450 2    50   ~ 0
+R4
+$Comp
+L Mechanical:MountingHole LOGO5
+U 1 1 5F1A21B2
+P 10700 10250
+F 0 "LOGO5" H 10950 10300 50  0000 C CNN
+F 1 "OSHW" H 11050 10200 50  0000 C CNN
+F 2 "josh-logos:OSHW_Logo_3.6x3.6_F.Mask" H 10700 10250 50  0001 C CNN
+F 3 "~" H 10700 10250 50  0001 C CNN
+	1    10700 10250
+	1    0    0    -1
+$EndComp
 $EndSCHEMATC

Commit message: designs off to fab
Parts:
- added C28, C32, C34: 1u, Capacitor_SMD:C_0603_1608Metric, symbol Device:C
- added C36, C38, C40: 100n, Capacitor_SMD:C_0603_1608Metric, symbol Device:C
Connections:
- net +3V3: now also C28.1, C32.1, C34.1, C36.1, C38.1, C40.1
- net GND: now also C28.2, C32.2, C34.2, C36.2, C38.2, C40.2
Other:
- note added: "Matrix"
- moved on the sheet: C48, C49, U3
