File: hardware/1.0/Hub20.sch (KiCad schematic (older format))
At the start: 149 parts, among them J1 USB_C_Receptacle_USB2.0, Q1 DTC123J, Q2 BSS138, SW1 EVQPUL, SW10 MX_RGB, SW11 MX_RGB, SW12 MX_RGB, SW13 EC11, SW14 MX_RGB, SW15 MX_RGB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

Commit message: add mechanicals
Parts:
- F1: Substitue Allowed? Y - 500mA hold / 1A trip -> Y - 1A hold / >1.5A trip
Changed lines of the file:
@@
 F 7 "Littelfuse" H 2850 1500 50  0001 C CNN "Manufacturer"
 F 8 "" H 2850 1500 50  0001 C CNN "Notes"
-F 9 "Y - 500mA hold / 1A trip" H 2850 1500 50  0001 C CNN "Substitue Allowed?"
+F 9 "Y - 1A hold / >1.5A trip" H 2850 1500 50  0001 C CNN "Substitue Allowed?"
 	1    2850 1500
 	0    1    1    0
