File: hardware/1.0/usb.sch (KiCad schematic (older format))
At the start: 34 parts, among them J2 USB_C_Receptacle_USB2.0, J3 USB_C_Receptacle_USB2.0, J4 USB_C_Receptacle_USB2.0, U5 CY7C65632-28LTXCT, U6 USBLC6-2SC6, U7 USBLC6-2SC6, U8 USBLC6-2SC6, Y2 12MHz

Commit message: add mechanicals
Parts:
- F2, F3, F4: Substitue Allowed? Y - 200mA hold / 500mA trip -> Y - 500mA hold / 1A trip
Changed lines of the file:
@@
 F 7 "Littelfuse" H 6700 1200 50  0001 C CNN "Manufacturer"
 F 8 "" H 6700 1200 50  0001 C CNN "Notes"
-F 9 "Y - 200mA hold / 500mA trip" H 6700 1200 50  0001 C CNN "Substitue Allowed?"
+F 9 "Y - 500mA hold / 1A trip" H 6700 1200 50  0001 C CNN "Substitue Allowed?"
 	1    6700 1200
 	0    1    1    0
@@
 F 7 "Littelfuse" H 8700 3375 50  0001 C CNN "Manufacturer"
 F 8 "" H 8700 3375 50  0001 C CNN "Notes"
-F 9 "Y - 200mA hold / 500mA trip" H 8700 3375 50  0001 C CNN "Substitue Allowed?"
+F 9 "Y - 500mA hold / 1A trip" H 8700 3375 50  0001 C CNN "Substitue Allowed?"
 	1    8700 3375
 	0    1    1    0
@@
 F 7 "Littelfuse" H 6300 4600 50  0001 C CNN "Manufacturer"
 F 8 "" H 6300 4600 50  0001 C CNN "Notes"
-F 9 "Y - 200mA hold / 500mA trip" H 6300 4600 50  0001 C CNN "Substitue Allowed?"
+F 9 "Y - 500mA hold / 1A trip" H 6300 4600 50  0001 C CNN "Substitue Allowed?"
 	1    6300 4600
 	0    1    1    0
