File: hardware/1.0.1/Hub20.kicad_pcb (KiCad board)
At the start: 2 copper layers, 89 x 124 mm, 183 parts, among them J1 USB_C_Receptacle_USB2.0, J2 USB_C_Receptacle_USB2.0, J3 USB_C_Receptacle_USB2.0, J4 USB_C_Receptacle_USB2.0, Q1 DTC123J, Q2 BSS138, SW1 EVQPUL, SW10 MX_RGB, SW11 MX_RGB, SW12 MX_RGB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

Commit message: update pcb for production
Parts:
- moved FB5 0.15 mm to (174.7, 46.0), turned to 180 degrees
Routing:
- net +5V: track 121.3 -> 122.8 mm
- net Net-(F4-Pad2): track 2.50 -> 1.99 mm
- net /R5: track 111.2 -> 111.7 mm
